File: camboard/camboard.sch (KiCad schematic (older format))
At the start: 61 parts, among them J1 USB_microB_2040002-1, J2 Micro_SD_Card, J3 PPTC102LFBN-RC, J4 Conn_ARM_JTAG_SWD_20, J5 GS2, J6 Conn_02x25_Row_Letter_First, SW1 SW_DPDT_x2, SW2 SW_Push, SW3 SW_Push, SW4 SW_DPDT_x2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

Commit message: Fixed oscillator symbol
Parts:
- removed Y1: SG-310SCN, Crystals:Crystal_SMD_3225-4pin_3.2x2.5mm, symbol Crystal_GND23
- added Y1: SG-310SCN, Crystals:Crystal_SMD_3225-4pin_3.2x2.5mm, symbol oscillator
Connections:
- wire segments 121 -> 163
Other:
- note removed: "??? Symbol"
- moved on the sheet: C6, C7, R12, R13, R14, U1B, Y2

Commit message: Finished schematic
Parts:
- removed C10, C11, C12, C13, C14, C9: 100nF, Capacitors_SMD:C_0603, symbol C
- added Cp2, Cp3, Cp4, Cp5, Cp6, Cp7: 100nF, Capacitors_SMD:C_0603, symbol C
- renumbered C2 to Ca2, C8 to Cp1
Connections:
- net labels added: CLK
- net labels removed: OSC25M

Commit message: Fixed some footprints
Parts:
- J6: footprint Pin_Headers:Pin_Header_Straight_2x25_Pitch2.54mm -> Socket_Strips:Socket_Strip_Straight_2x25_Pitch2.54mm
- SW1, SW5: footprint Buttons_Switches_THT:SW_CuK_JS202011CQN_DPDT_Straight -> DPDT_switch:JS202011SCQN
Connections:
- wire segments 163 -> 120
Changed lines of the file:
@@
 F 0 "SW1" H 3400 7350 50  0000 C CNN
 F 1 "SW_DPDT_x2" H 3650 6800 50  0000 C CNN
-F 2 "Buttons_Switches_THT:SW_CuK_JS202011CQN_DPDT_Straight" H 3500 7275 50  0001 C CNN
+F 2 "DPDT_switch:JS202011SCQN" H 3500 7275 50  0001 C CNN
 F 3 "" H 3400 7195 50  0001 C CNN
 	1    3400 7025
@@
 F 0 "J6" H 10025 5625 50  0000 C CNN
 F 1 "Conn_02x25_Row_Letter_First" V 10200 3625 50  0000 C CNN
-F 2 "Pin_Headers:Pin_Header_Straight_2x25_Pitch2.54mm" H 9975 4625 50  0001 C CNN
+F 2 "Socket_Strips:Socket_Strip_Straight_2x25_Pitch2.54mm" H 9975 4625 50  0001 C CNN
 F 3 "" H 9975 4625 50  0001 C CNN
 	1    9975 4625
@@
 F 0 "SW5" H 6475 7725 50  0000 C CNN
 F 1 "SW_DPDT_x2" H 6725 7225 50  0000 C CNN
-F 2 "Buttons_Switches_THT:SW_CuK_JS202011CQN_DPDT_Straight" H 6575 7700 50  0001 C CNN
+F 2 "DPDT_switch:JS202011SCQN" H 6575 7700 50  0001 C CNN
 F 3 "" H 6475 7620 50  0001 C CNN
 	1    6475 7450
@@
 $EndComp
 Wire Wire Line
-	10850 1225 10850 1425
-Wire Wire Line
-	10850 1425 10850 1650
+	10850 1225 10850 1650
 Wire Wire Line
 	10550 1425 10550 1650
@@
 	10200 1325 10200 1425
 Wire Wire Line
-	2375 1475 2450 1475
-Wire Wire Line
-	2450 1475 3175 1475
+	2375 1475 3175 1475
 Wire Wire Line
 	2450 1475 2450 1100
 Wire Wire Line
-	2375 1575 2600 1575
-Wire Wire Line
-	2600 1575 3175 1575
+	2375 1575 3175 1575
 Wire Wire Line
 	2600 1575 2600 1100
 Wire Wire Line
-	2375 1675 2750 1675
-Wire Wire Line
-	2750 1675 3175 1675
+	2375 1675 3175 1675
 Wire Wire Line
 	2750 1675 2750 1100
 Wire Wire Line
-	2375 1775 2900 1775
-Wire Wire Line
-	2900 1775 3175 1775
+	2375 1775 3175 1775
 Wire Wire Line
 	2900 1775 2900 1100
 Wire Wire Line
-	2375 1875 3050 1875
-Wire Wire Line
-	3050 1875 3175 1875
+	2375 1875 3175 1875
 Wire Wire Line
 	3050 1875 3050 1100
@@
 Connection ~ 3050 1875
 Wire Wire Line
-	2450 800  2600 800
-Wire Wire Line
-	2600 800  2750 800
-Wire Wire Line
-	2750 800  2900 800
-Wire Wire Line
-	2900 800  3050 800
+	2450 800  3050 800
 Connection ~ 2600 800
 Connection ~ 2750 800
 Connection ~ 2900 800
 Wire Wire Line
-	4700 850  4750 850
-Wire Wire Line
-	4750 850  4800 850
+	4700 850  4800 850
 Connection ~ 4750 850
 Wire Wire Line
@@
 	5800 1450 5800 2225
 Wire Wire Line
-	2475 6125 3150 6125
-Wire Wire Line
-	3150 6125 3250 6125
-Wire Wire Line
-	3250 6125 3350 6125
+	2475 6125 3350 6125
 Connection ~ 3250 6125
 Wire Wire Line
@@
 	4775 7450 4725 7450
 Wire Wire Line
-	4650 7025 4650 7050
-Wire Wire Line
-	4650 7050 4650 7150
-Wire Wire Line
-	4650 7150 4650 7250
+	4650 7025 4650 7250
 Wire Wire Line
 	4650 7050 4775 7050
@@
 Connection ~ 4650 7250
 Wire Wire Line
-	700  7600 900  7600
-Wire Wire Line
-	900  7600 1100 7600
-Wire Wire Line
-	1100 7600 1300 7600
-Wire Wire Line
-	1300 7600 1500 7600
-Wire Wire Line
-	1500 7600 1700 7600
-Wire Wire Line
-	1700 7600 1900 7600
-Wire Wire Line
-	1900 7600 2100 7600
-Wire Wire Line
-	2100 7600 2300 7600
-Wire Wire Line
-	2300 7600 2500 7600
+	700  7600 2500 7600
 Connection ~ 900  7600
 Connection ~ 1100 7600
@@
 Connection ~ 2300 7600
 Wire Wire Line
-	550  7300 700  7300
-Wire Wire Line
-	700  7300 900  7300
-Wire Wire Line
-	900  7300 1100 7300
-Wire Wire Line
-	1100 7300 1300 7300
-Wire Wire Line
-	1300 7300 1500 7300
-Wire Wire Line
-	1500 7300 1700 7300
-Wire Wire Line
-	1700 7300 1900 7300
-Wire Wire Line
-	1900 7300 2100 7300
-Wire Wire Line
-	2100 7300 2300 7300
-Wire Wire Line
-	2300 7300 2500 7300
+	550  7300 2500 7300
 Connection ~ 700  7300
 Connection ~ 900  7300
@@
 	6325 7150 6325 7050
 Wire Wire Line
-	6100 6750 6325 6750
-Wire Wire Line
-	6325 6750 6525 6750
+	6100 6750 6525 6750
 Connection ~ 6325 6750
 Wire Wire Line
@@
 	5975 7350 6200 7350
 Wire Wire Line
-	2475 5625 2475 5675
-Wire Wire Line
-	2475 5675 2475 5725
-Wire Wire Line
-	2475 5725 2475 5825
+	2475 5625 2475 5825
 Wire Wire Line
 	5625 5325 5550 5325
@@
 	5625 5025 5625 5325
 Wire Wire Line
-	3600 7325 3975 7325
-Wire Wire Line
-	3975 7325 4375 7325
+	3600 7325 4375 7325
 Connection ~ 4775 7350
 Connection ~ 3975 7325
 Wire Wire Line
-	4275 7025 4325 7025
-Wire Wire Line
-	4325 7025 4375 7025
-Wire Wire Line
-	4375 7025 4650 7025
+	4275 7025 4650 7025
 Connection ~ 4325 7025
 Connection ~ 4375 7025
@@
 	2800 7750 2800 6550
 Wire Wire Line
-	800  6075 900  6075
-Wire Wire Line
-	900  6075 1000 6075
-Wire Wire Line
-	1000 6075 1100 6075
-Wire Wire Line
-	1100 6075 1200 6075
-Wire Wire Line
-	1200 6075 1300 6075
-Wire Wire Line
-	1300 6075 1375 6075
+	800  6075 1375 6075
 Wire Wire Line
 	1375 6075 1375 6125
@@
 	7700 3925 8275 3925
 Wire Wire Line
-	1800 4850 1925 4850
-Wire Wire Line
-	1925 4850 2050 4850
+	1800 4850 2050 4850
 Wire Wire Line
 	1800 4850 1800 4975

Commit message: 2x1->1x2
Parts:
- removed J6: Conn_02x25_Row_Letter_First, Socket_Strips:Socket_Strip_Straight_2x25_Pitch2.54mm, symbol Conn_02x25_Row_Letter_First
- added J6, J7: Conn_01x25_Female, Pin_Headers:Pin_Header_Straight_1x25_Pitch2.54mm, symbol Conn_01x25_Female

Commit message: properly updated switch
Parts:
- SW1, SW4, SW5: symbol SW_DPDT_x2 -> SW_DPDT_x2-RESCUE-camboard
Changed lines of the file:
@@
 $EndComp
 $Comp
-L SW_DPDT_x2 SW1
+L SW_DPDT_x2-RESCUE-camboard SW1
 U 1 1 59CBC80C
 P 3400 7025
@@
 $EndComp
 $Comp
-L SW_DPDT_x2 SW4
+L SW_DPDT_x2-RESCUE-camboard SW4
 U 1 1 59CF7B5F
 P 10850 4325
@@
 ??? Interupts\n
 $Comp
-L SW_DPDT_x2 SW5
+L SW_DPDT_x2-RESCUE-camboard SW5
 U 1 1 59D83FE7
 P 6475 7450
@@
 $EndComp
 $Comp
-L SW_DPDT_x2 SW1
+L SW_DPDT_x2-RESCUE-camboard SW1
 U 2 1 59D847D4
 P 3400 7025
@@
 $EndComp
 $Comp
-L SW_DPDT_x2 SW5
+L SW_DPDT_x2-RESCUE-camboard SW5
 U 2 1 59D84B7E
 P 6475 7450
@@
 $EndComp
 $Comp
-L SW_DPDT_x2 SW4
+L SW_DPDT_x2-RESCUE-camboard SW4
 U 2 1 59D85D34
 P 10850 4325

Commit message: remove cp7
Parts:
- removed Cp7: 100nF, Capacitors_SMD:C_0603, symbol C
Changed lines of the file:
@@
 Connection ~ 2100 7600
 Connection ~ 2300 7600
-Wire Wire Line
-	550  7300 2500 7300
 Connection ~ 700  7300
 Connection ~ 900  7300
@@
 $EndComp
 $Comp
-L C Cp7
-U 1 1 59D9FF2F
-P 2500 7450
-F 0 "Cp7" H 2525 7550 50  0000 L CNN
-F 1 "100nF" V 2525 7050 50  0000 L CNN
-F 2 "Capacitors_SMD:C_0603" H 2538 7300 50  0001 C CNN
-F 3 "" H 2500 7450 50  0001 C CNN
-	1    2500 7450
-	-1   0    0    1
-$EndComp
-$Comp
 L Conn_01x25_Female J7
 U 1 1 59D82062
@@
 	-1   0    0    1
 $EndComp
+Wire Wire Line
+	2300 7300 550  7300
 $EndSCHEMATC

Commit message: Finished(ish) placing components
Parts:
- SW1, SW4, SW5: symbol SW_DPDT_x2-RESCUE-camboard -> SW_DPDT_x2
Changed lines of the file:
@@
 EESchema Schematic File Version 2
-LIBS:camboard-rescue
 LIBS:stm32-v2
 LIBS:components
@@
 $EndComp
 $Comp
-L SW_DPDT_x2-RESCUE-camboard SW1
+L SW_DPDT_x2 SW1
 U 1 1 59CBC80C
 P 3400 7025
@@
 $EndComp
 $Comp
-L SW_DPDT_x2-RESCUE-camboard SW4
+L SW_DPDT_x2 SW4
 U 1 1 59CF7B5F
 P 10850 4325
@@
 ??? Interupts\n
 $Comp
-L SW_DPDT_x2-RESCUE-camboard SW5
+L SW_DPDT_x2 SW5
 U 1 1 59D83FE7
 P 6475 7450
@@
 $EndComp
 $Comp
-L SW_DPDT_x2-RESCUE-camboard SW1
+L SW_DPDT_x2 SW1
 U 2 1 59D847D4
 P 3400 7025
@@
 $EndComp
 $Comp
-L SW_DPDT_x2-RESCUE-camboard SW5
+L SW_DPDT_x2 SW5
 U 2 1 59D84B7E
 P 6475 7450
@@
 $EndComp
 $Comp
-L SW_DPDT_x2-RESCUE-camboard SW4
+L SW_DPDT_x2 SW4
 U 2 1 59D85D34
 P 10850 4325

Commit message: fixed jtag
Parts:
- J4: footprint Pin_Headers:Pin_Header_Straight_2x05_Pitch2.54mm -> Pin_Headers:Pin_Header_Straight_2x10_Pitch2.54mm
Changed lines of the file:
@@
 F 0 "J4" H 4400 900 50  0000 R CNN
 F 1 "Conn_ARM_JTAG_SWD_20" H 5275 575 50  0000 R BNN
-F 2 "Pin_Headers:Pin_Header_Straight_2x05_Pitch2.54mm" H 5250 600 50  0001 L TNN
+F 2 "Pin_Headers:Pin_Header_Straight_2x10_Pitch2.54mm" H 5250 600 50  0001 L TNN
 F 3 "" V 4450 400 50  0001 C CNN
 	1    4800 1650
