File: camboard/camboard.kicad_pcb (KiCad board)
At the start: 2 copper layers, 76.2 x 76.2 mm, 60 parts, among them J1 USB_microB_2040002-1, J2 Micro_SD_Card, J3 PPTC102LFBN-RC, J4 Conn_ARM_JTAG_SWD_20, J5 GS2, J6 Conn_01x25_Female, J7 Conn_01x25_Female, SW1 SW_DPDT_x2, SW2 SW_Push, SW3 SW_Push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

Commit message: Pre-autoroute
Parts:
- moved R12 0.74 mm to (59.7, 97.2), turned to 180 degrees
Routing:
- net Net-(J6-Pad21): track 0.00 -> 50.2 mm
- net Net-(J6-Pad20): track 0.00 -> 47.8 mm
- net Net-(J6-Pad19): track 0.00 -> 41.7 mm
- net Net-(J6-Pad22): track 0.00 -> 40.5 mm
- net Net-(J6-Pad18): track 0.00 -> 39.5 mm
- net /NRST: track 0.00 -> 37.8 mm, vias 0 -> 2
- net Net-(J6-Pad5): track 0.00 -> 35.2 mm
- net Net-(J6-Pad17): track 0.00 -> 34.5 mm
- net Net-(R13-Pad1): track 0.00 -> 34.1 mm
- net Net-(R14-Pad1): track 0.00 -> 33.1 mm
- net Net-(J6-Pad16): track 0.00 -> 31.5 mm
- net Net-(R12-Pad2): track 0.00 -> 20.2 mm
- net Net-(C7-Pad2): track 0.00 -> 9.97 mm
- net Net-(C6-Pad1): track 0.00 -> 7.47 mm
- net Net-(R12-Pad1): track 0.00 -> 4.02 mm

Commit message: autoroute
Routing:
- net GND: track 309.4 -> 476.8 mm, vias 6 -> 8
- net +3V3: track 225.8 -> 346.4 mm, vias 8 -> 13
- net Net-(J3-Pad7): track 0.00 -> 104.8 mm, vias 0 -> 1
- net /NRST: track 37.8 -> 108.2 mm
- net Net-(J2-Pad5): track 0.00 -> 68.1 mm, vias 0 -> 2
- net /DCMI_D5: track 0.00 -> 65.4 mm, vias 0 -> 1
- net /DCMI_PWDN: track 0.00 -> 63.4 mm, vias 0 -> 3
- net Net-(J3-Pad3): track 0.00 -> 59.9 mm, vias 0 -> 2
- net Net-(J3-Pad4): track 0.00 -> 48.5 mm, vias 0 -> 3
- net Net-(J6-Pad24): track 0.00 -> 48.0 mm, vias 0 -> 2
- net Net-(J2-Pad1): track 19.9 -> 66.9 mm, vias 0 -> 2
- net Net-(J7-Pad6): track 0.00 -> 47.0 mm
- net Net-(J4-Pad13): track 0.00 -> 46.7 mm, vias 0 -> 1
- net Net-(J6-Pad23): track 0.00 -> 46.3 mm, vias 0 -> 2
- net Net-(J4-Pad3): track 0.00 -> 45.0 mm, vias 0 -> 1
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
Commit message: Final autorouting
Routing:
- net +3V3: track 346.4 -> 339.8 mm
- net Net-(J2-Pad5): track 68.1 -> 64.4 mm
- net Net-(J3-Pad4): track 48.5 -> 51.5 mm
- net Net-(J3-Pad3): track 59.9 -> 59.0 mm
- net GND: track 476.8 -> 476.1 mm

Commit message: updated pcb
Routing:
- net Net-(R13-Pad1): track 34.1 -> 34.7 mm

Commit message: Fixed some silly traces
Routing:
- net GND: track 476.1 -> 482.2 mm
- net Net-(J6-Pad22): track 40.5 -> 41.1 mm
- net Net-(J3-Pad7): track 104.8 -> 105.3 mm

Commit message: More changes
Routing:
- net GND: track 482.2 -> 482.4 mm, vias 8 -> 10
- net Net-(J7-Pad3): vias 1 -> 0
- added copper zone on B.Cu, net GND
Changed lines of the file:
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@@
     (thickness 1.6)
     (drawings 7)
-    (tracks 1368)
+    (tracks 1370)
     (zones 0)
     (modules 60)
@@
   (gr_line (start 114.3 38.1) (end 114.3 114.3) (layer Edge.Cuts) (width 0.15))
   (gr_line (start 38.1 38.1) (end 114.3 38.1) (layer Edge.Cuts) (width 0.15))
+  (via (at 94.852 47.752) (size 0.5842) (drill 0.381) (layers F.Cu B.Cu) (net 1))
+  (segment (start 52.156 98.13547) (end 47.101083 103.190387) (width 0.4) (layer F.Cu) (net 1))
+  (segment (start 45.515 103.505) (end 46.78647 103.505) (width 0.4) (layer F.Cu) (net 1))
+  (via (at 46.808984 103.482486) (size 0.5842) (drill 0.381) (layers F.Cu B.Cu) (net 1))
+  (segment (start 46.78647 103.505) (end 46.808984 103.482486) (width 0.4) (layer F.Cu) (net 1))
+  (segment (start 47.101083 103.190387) (end 46.808984 103.482486) (width 0.4) (layer F.Cu) (net 1))
+  (segment (start 52.156 86.36) (end 52.156 98.13547) (width 0.4) (layer F.Cu) (net 1))
   (segment (start 79.311389 88.671564) (end 87.701574 80.281379) (width 0.4) (layer B.Cu) (net 1))
   (segment (start 87.701574 80.281379) (end 87.701574 77.393223) (width 0.4) (layer B.Cu) (net 1))
@@
   (segment (start 53.1811 81.2869) (end 62.4703 81.2869) (width 0.4) (layer F.Cu) (net 1))
   (segment (start 52.156 86.36) (end 52.156 83.312) (width 0.4) (layer F.Cu) (net 1) (status 30))
-  (segment (start 46.365 103.505) (end 52.156 97.714) (width 0.4) (layer F.Cu) (net 1))
-  (segment (start 45.515 103.505) (end 46.365 103.505) (width 0.4) (layer F.Cu) (net 1) (status 10))
-  (segment (start 52.156 97.714) (end 52.156 86.36) (width 0.4) (layer F.Cu) (net 1) (status 20))
   (segment (start 46.287401 105.527401) (end 45.515 104.755) (width 0.4) (layer F.Cu) (net 1))
   (segment (start 51.367401 112.337153) (end 50.742153 112.962401) (width 0.4) (layer F.Cu) (net 1))
@@
   (segment (start 71.068699 82.5781) (end 71.0878 82.5781) (width 0.1524) (layer F.Cu) (net 77) (status 30))
   (segment (start 71.0877 82.5781) (end 71.068699 82.5781) (width 0.1524) (layer F.Cu) (net 77) (status 30))
-  (segment (start 59.575498 86.728502) (end 58.578949 86.728502) (width 0.1524) (layer F.Cu) (net 78))
+  (segment (start 68.2593 79.7496) (end 68.2593 79.7497) (width 0.1524) (layer F.Cu) (net 78))
   (segment (start 65.9533 80.3507) (end 59.575498 86.728502) (width 0.1524) (layer F.Cu) (net 78))
-  (segment (start 52.889422 109.035578) (end 50.165 111.76) (width 0.1524) (layer F.Cu) (net 78) (status 20))
-  (segment (start 52.889422 93.414578) (end 52.889422 109.035578) (width 0.1524) (layer F.Cu) (net 78))
-  (segment (start 58.016621 88.287379) (end 52.889422 93.414578) (width 0.1524) (layer F.Cu) (net 78))
+  (segment (start 53.006169 108.918831) (end 51.014999 110.910001) (width 0.1524) (layer F.Cu) (net 78))
+  (segment (start 53.006169 93.297831) (end 53.006169 108.918831) (width 0.1524) (layer F.Cu) (net 78))
+  (segment (start 58.578949 86.728502) (end 58.016621 87.29083) (width 0.1524) (layer F.Cu) (net 78))
+  (segment (start 68.2593 79.7497) (end 67.6583 80.3507) (width 0.1524) (layer F.Cu) (net 78))
+  (segment (start 51.014999 110.910001) (end 50.165 111.76) (width 0.1524) (layer F.Cu) (net 78))
   (segment (start 58.016621 87.29083) (end 58.016621 88.287379) (width 0.1524) (layer F.Cu) (net 78))
-  (segment (start 68.2593 79.7497) (end 67.6583 80.3507) (width 0.1524) (layer F.Cu) (net 78) (status 10))
+  (segment (start 58.016621 88.287379) (end 53.006169 93.297831) (width 0.1524) (layer F.Cu) (net 78))
   (segment (start 67.6583 80.3507) (end 65.9533 80.3507) (width 0.1524) (layer F.Cu) (net 78))
-  (segment (start 68.2593 79.7496) (end 68.2593 79.7497) (width 0.1524) (layer F.Cu) (net 78) (status 30))
-  (segment (start 58.578949 86.728502) (end 58.016621 87.29083) (width 0.1524) (layer F.Cu) (net 78))
+  (segment (start 59.575498 86.728502) (end 58.578949 86.728502) (width 0.1524) (layer F.Cu) (net 78))
+  (segment (start 52.584611 106.800389) (end 52.584611 91.423989) (width 0.1524) (layer F.Cu) (net 79))
+  (segment (start 52.584611 91.423989) (end 57.6486 86.36) (width 0.1524) (layer F.Cu) (net 79))
+  (segment (start 47.625 111.76) (end 52.584611 106.800389) (width 0.1524) (layer F.Cu) (net 79))
   (segment (start 57.6486 86.36) (end 57.73479 86.36) (width 0.1524) (layer F.Cu) (net 79) (status 30))
   (segment (start 59.2228 84.34561) (end 59.48599 84.6088) (width 0.1524) (layer B.Cu) (net 79))
@@
   (segment (start 59.2228 78.4049) (end 59.2228 84.34561) (width 0.1524) (layer B.Cu) (net 79))
   (via (at 59.48599 84.6088) (size 0.5842) (drill 0.381) (layers F.Cu B.Cu) (net 79))
-  (segment (start 52.584611 106.800389) (end 52.584611 91.423989) (width 0.1524) (layer F.Cu) (net 79))
-  (segment (start 52.584611 91.423989) (end 57.6486 86.36) (width 0.1524) (layer F.Cu) (net 79) (status 20))
-  (segment (start 47.625 111.76) (end 52.584611 106.800389) (width 0.1524) (layer F.Cu) (net 79) (status 10))
   (via (at 59.2228 78.4049) (size 0.5842) (layers F.Cu B.Cu) (net 79))
   (segment (start 57.888 86.36) (end 57.6486 86.36) (width 0.1524) (layer F.Cu) (net 79) (status 30))
@@
   (segment (start 54.84 47.752) (end 56.0586 47.752) (width 0.25) (layer F.Cu) (net 82) (status 10))
   (segment (start 71.0878 69.9915) (end 71.0877 69.9916) (width 0.1524) (layer F.Cu) (net 82) (status 30))
-  (via (at 53.5745 45.0612) (size 0.5842) (layers F.Cu B.Cu) (net 83))
-  (segment (start 52.9902 45.0612) (end 53.5745 45.0612) (width 0.1524) (layer B.Cu) (net 83))
-  (segment (start 48.7039 40.7749) (end 52.9902 45.0612) (width 0.1524) (layer B.Cu) (net 83))
-  (segment (start 48.7039 40.64) (end 48.7039 40.7749) (width 0.1524) (layer B.Cu) (net 83))
-  (segment (start 70.8407 69.0374) (end 71.4413 69.638) (width 0.1524) (layer F.Cu) (net 83) (status 20))
-  (segment (start 70.8407 61.9902) (end 70.8407 69.0374) (width 0.1524) (layer F.Cu) (net 83))
+  (segment (start 47.625 40.64) (end 48.56867 40.64) (width 0.1524) (layer F.Cu) (net 83))
+  (segment (start 48.56867 40.64) (end 52.98987 45.0612) (width 0.1524) (layer F.Cu) (net 83))
+  (segment (start 52.98987 45.0612) (end 53.9117 45.0612) (width 0.1524) (layer F.Cu) (net 83))
   (segment (start 53.9117 45.0612) (end 70.8407 61.9902) (width 0.1524) (layer F.Cu) (net 83))
-  (segment (start 53.5745 45.0612) (end 53.9117 45.0612) (width 0.1524) (layer F.Cu) (net 83))
-  (segment (start 47.625 40.64) (end 48.7039 40.64) (width 0.1524) (layer B.Cu) (net 83) (status 10))
+  (segment (start 70.8407 61.9902) (end 70.8407 69.0374) (width 0.1524) (layer F.Cu) (net 83))
+  (segment (start 70.8407 69.0374) (end 71.4413 69.638) (width 0.1524) (layer F.Cu) (net 83))
   (segment (start 50.165 40.64) (end 50.165 41.7189) (width 0.1524) (layer F.Cu) (net 84) (status 10))
   (segment (start 72.502 68.5773) (end 71.8098 67.885) (width 0.1524) (layer F.Cu) (net 84) (status 10))
@@
       )
     )
+  )
+  (zone (net 1) (net_name GND) (layer B.Cu) (hatch edge 0.508)
+    (connect_pads (clearance 0.508))
+    (min_thickness 0.254)
+    (fill yes (arc_segments 16) (thermal_gap 0.508) (thermal_bridge_width 0.508))
+    (polygon
+      (pts
+        (xy 37.9984 38.0492) (xy 114.2492 38.1) (xy 114.2492 114.2492) (xy 37.9984 114.3) (xy 37.9984 38.2524)
+        (xy 37.9984 38.2524)
+      )
+    )

Commit message: report-version
Parts:
- moved R22 9.53 mm to (61.0, 54.4)
- moved C17 2.33 mm to (93.2, 47.8), turned to 180 degrees
Routing:
- net Net-(J7-Pad2): track 42.5 -> 71.5 mm
- net Net-(R22-Pad1): track 8.60 -> 16.2 mm
- net GND: track 482.4 -> 477.7 mm, vias 10 -> 9
- net Net-(C17-Pad1): track 15.7 -> 12.7 mm
- net /DCMI_D5: track 65.4 -> 64.6 mm
Other:
- board text added: "Eric & Jamie"
- board text added: "GND"
- board text added: "MCO"
- board text added: "PA1 PE2 PE3 PC13 PC0 PC1 PC2 PC3 PA2 PA3 PA5 PA7 PC4 PC5 PB0 PB1 PB2 PE7 PE8 PE9 PE10"
- board text added: "PA11"
- board text added: "PA12"
- board text added: "PB12"
- board text added: "PB13"
- board text added: "PB14"
- board text added: "PB15"
- board text added: "PD0"
- board text added: "PD1"
- board text added: "PD10"
- board text added: "PD13"
- board text added: "PD14"
- board text added: "PD15"
- board text added: "PD4"
- board text added: "PD5"
- board text added: "PD7"
- board text added: "PE11"
- board text added: "PE12"
- board text added: "PE13"
- board text added: "PE14"
- board text added: "PE15"
- board text added: "USB"
- board text added: "VIN"

Commit message: beautifying
Parts:
- J3, J4: footprint Pin_Headers:Pin_Header_Straight_2x10_Pitch2.54mm -> 2x10_Female_Header:Socket_Strip_Straight_2x10_Pitch2.54mm
- J6, J7: footprint Pin_Headers:Pin_Header_Straight_1x25_Pitch2.54mm -> Socket_Strips:Socket_Strip_Straight_1x25_Pitch2.54mm
- moved J2 2.54 mm to (100.7, 96.1)
Connections:
- J3 pad 17: (no net) -> Net-(J3-Pad17)
- J3 pad 18: (no net) -> Net-(J3-Pad18)
- J6 pad 1: (no net) -> Net-(J6-Pad1)
- J6 pad 2: (no net) -> Net-(J6-Pad2)
- J6 pad 3: (no net) -> Net-(J6-Pad3)
- U1 pad 13: (no net) -> Net-(U1-Pad13)
- U1 pad 6: (no net) -> Net-(U1-Pad6)
- U1 pad 63: (no net) -> Net-(U1-Pad63)
- U1 pad 64: (no net) -> Net-(U1-Pad64)
- U1 pad 87: (no net) -> Net-(U1-Pad87)
- U1 pad 91: (no net) -> Net-(U1-Pad91)
- U1 pad 92: (no net) -> Net-(U1-Pad92)
- U1 pad 95: (no net) -> Net-(U1-Pad95)
- U1 pad 96: (no net) -> Net-(U1-Pad96)
- U3 pad 10: (no net) -> Net-(U3-Pad10)
- U3 pad 15: (no net) -> Net-(U3-Pad15)
- U3 pad 16: (no net) -> Net-(U3-Pad16)
Other:
- outline, holes or cut-outs redrawn
- board text added: "PD7 PD5 PD4 PD1 PD0 PA12 PA11 MCO PD15 PD14 PD13 PD10 PB15 PB14 PB13 PB12 PE15 PE14 PE13 PE12 PE11 VIN USB GND GND"
- board text removed: "GND"
- board text removed: "MCO"
- board text removed: "PA11"
- board text removed: "PA12"
- board text removed: "PB12"
- board text removed: "PB13"
- board text removed: "PB14"
- board text removed: "PB15"
- board text removed: "PD0"
- board text removed: "PD1"
- board text removed: "PD10"
- board text removed: "PD13"
- board text removed: "PD14"
- board text removed: "PD15"
- board text removed: "PD4"
- board text removed: "PD5"
- board text removed: "PD7"
- board text removed: "PE11"
- board text removed: "PE12"
- board text removed: "PE13"
- board text removed: "PE14"
- board text removed: "PE15"
- board text removed: "USB"
- board text removed: "VIN"
